Commit message: Prune unused meshes and unify left/right thumb convention
Housekeeping pass on the description package. The body model and all
finger geometry are untouched; only the right thumb's naming and the
thumb joint limits change.

Remove 63 unused STL meshes (22 MB, package 96 MB -> 74 MB):
- 52 meshes of the older Unitree Inspire hand (link11_L..link22_R,
  L/R_*_proximal/intermediate/distal, L/R_hand_base_link), left over
  from copying Unitree's meshes/ wholesale
- 8 parallel ankle-mechanism meshes (*_ankle_A/B_link, *_ankle_A/B_rod_link)
- 4 body leftovers (left/right_hand_link, right_ankle_link, right_pitch_link)
- hand_left/flange.STL

Unify the thumb naming so both hands use the same joint and link names,
adopting the left hand's convention (swing + 1..3):
  right_thumb_1 -> right_thumb_swing   (abduction, actuated)
  right_thumb_2 -> right_thumb_1       (flexion, actuated)
  right_thumb_3 -> right_thumb_2       (mimic x0.40)
  right_thumb_4 -> right_thumb_3       (mimic x0.60)
Applied to the xacro, the flat Isaac URDF, the RViz config, the README
and the four STL files, so hand_left/ and hand_right/ now hold the same
13 filenames. The 24 hand joints are identical once the left_/right_
prefix is stripped.

Unify the thumb joint limits across hands:
  *_thumb_swing_joint  [0, 1.7] / [0, 1.70]     -> [0, 1.70]
  *_thumb_1_joint      [0, 0.92] / [0.035, 0.90] -> [0, 0.92]
The right thumb's 0.035 lower bound made joint_state_publisher clamp it
to a different rest pose than the left. Both thumbs now start at 0; the
right thumb tip moves 2.50 mm and the mismatch against the mirrored left
drops from 21.55 mm to 20.89 mm.

Validated: XML well-formed (8/8), xacro expands (4/4), check_urdf clean
(3/3), loads in Pinocchio (njoints=52, nq=51, mass=61.8499 kg), limits
symmetric on 12/12 joint pairs, no dangling or unused mesh references.

Known issue, not addressed here: the thumbs are still not mirror images.
The four fingers match to 0.01-1.5 mm, but the thumb diverges from
*_thumb_1_joint onward (7.3 -> 18.0 -> 29.0 mm on the link centroids),
because its origin rpy is "1.5708 0 0.037536" on the left and
"1.5708 0 2.7925" on the right -- about 17 degrees off the mirror. Fixing
it means picking which side's vendor export is authoritative.

Co-Authored-By: Claude Opus 5 <noreply@anthropic.com>
Claude-Session: https://claude.ai/code/session_01WDAX8VZbrLhjdUkohUZLGo

File: urdf/h1_2_hands_isaac.urdf (robot description, URDF)
Before this commit: robot h1_2_with_inspire_hands, 58 links, 57 joints
Links:
- removed link right_thumb_4
- added link right_thumb_swing, mass 0.00115518743162309; collision mesh filename=package://h1_2_inspire_description/meshes/hand_right/right_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; visual mesh filename=package://h1_2_inspire_description/meshes/hand_right/right_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
- link right_thumb_1: mass 0.00115518743162309 -> 0.030
- link right_thumb_2: mass 0.030 -> 0.020
- link right_thumb_3: mass 0.020 -> 0.014
Joints:
- removed joint right_thumb_4_joint
- added joint right_thumb_swing_joint: type revolute, parent right_hand_base_link, child right_thumb_swing, origin xyz=-0.035227 -0.0908 -0.041956 rpy=0 0 0, axis 0 0 -1, limit lower=0 upper=1.70 effort=1 velocity=100
- joint right_thumb_1_joint: axis 0 0 -1 -> 0 0 1; limit lower=0 upper=1.7 effort=1 velocity=100 -> lower=0 upper=0.92 effort=1 velocity=100; origin xyz=-0.035227 -0.0908 -0.041956 rpy=0 0 0 -> xyz=-0.0063016 0.011924 0.003 rpy=1.5708 0 2.7925; parent right_hand_base_link -> right_thumb_swing
- joint right_thumb_2_joint: limit lower=0.035 upper=0.90 effort=1 velocity=100 -> lower=0 upper=3.14 effort=1 velocity=100; origin xyz=-0.0063016 0.011924 0.003 rpy=1.5708 0 2.7925 -> xyz=0.038292 0.014535 -0.0015 rpy=0 0 0
- joint right_thumb_3_joint: origin xyz=0.038292 0.014535 -0.0015 rpy=0 0 0 -> xyz=0.018189 0.012576 -0.0002 rpy=0 0 0

File: urdf/inspire_hand_right.urdf.xacro (robot description, xacro)
@@ -2,7 +2,7 @@
 <!-- Inspire RH56DFTP right hand — fragment included by combined and standalone files.
      Root link: right_hand_base_link
-     Actuated joints (6): right_thumb_1_joint, right_thumb_2_joint,
+     Actuated joints (6): right_thumb_swing_joint, right_thumb_1_joint,
        right_index_1_joint, right_middle_1_joint, right_ring_1_joint, right_little_1_joint
-     Mimic joints: right_thumb_3_joint (0.40×), right_thumb_4_joint (0.60×),
+     Mimic joints: right_thumb_2_joint (0.40×), right_thumb_3_joint (0.60×),
        right_index_2_joint (1.05×), right_middle_2_joint (1.05×),
        right_ring_2_joint (1.05×), right_little_2_joint (1.05×) -->
@@ -31,5 +31,5 @@
     </collision>
   </link>
-  <link name="right_thumb_1">
+  <link name="right_thumb_swing">
     <inertial>
       <origin xyz="-0.00178423179132727 0.000649410769092446 0.0048858931043441" rpy="0 0 0"/>
@@ -41,25 +41,25 @@
       <origin xyz="0 0 0" rpy="0 0 0"/>
       <geometry>
-        <mesh filename="package://h1_2_inspire_description/meshes/hand_right/right_thumb_1.STL"/>
-      </geometry>
-      <material name="">
-        <color rgba="1 1 1 1"/>
-      </material>
-    </visual>
-    <collision>
-      <origin xyz="0 0 0" rpy="0 0 0"/>
-      <geometry>
-        <mesh filename="package://h1_2_inspire_description/meshes/hand_right/right_thumb_1.STL"/>
-      </geometry>
-    </collision>
-  </link>
-  <joint name="right_thumb_1_joint" type="revolute">
+        <mesh filename="package://h1_2_inspire_description/meshes/hand_right/right_thumb_swing.STL"/>
+      </geometry>
+      <material name="">
+        <color rgba="1 1 1 1"/>
+      </material>
+    </visual>
+    <collision>
+      <origin xyz="0 0 0" rpy="0 0 0"/>
+      <geometry>
+        <mesh filename="package://h1_2_inspire_description/meshes/hand_right/right_thumb_swing.STL"/>
+      </geometry>
+    </collision>
+  </link>
+  <joint name="right_thumb_swing_joint" type="revolute">
     <origin xyz="-0.035227 -0.0908 -0.041956" rpy="0 0 0"/>
     <parent link="right_hand_base_link"/>
-    <child link="right_thumb_1"/>
+    <child link="right_thumb_swing"/>
     <axis xyz="0 0 -1"/>
-    <limit lower="0" upper="1.7" effort="1" velocity="100"/>
-  </joint>
-  <link name="right_thumb_2">
+    <limit lower="0" upper="1.70" effort="1" velocity="100"/>
+  </joint>
+  <link name="right_thumb_1">
     <inertial>
       <origin xyz="0.0161097484383394 0.0103028022975375 -0.00905330600289518" rpy="0 0 0"/>
@@ -71,25 +71,25 @@
       <origin xyz="0 0 0" rpy="0 0 0"/>
       <geometry>
-        <mesh filename="package://h1_2_inspire_description/meshes/hand_right/right_thumb_2.STL"/>
-      </geometry>
-      <material name="">
-        <color rgba="1 1 1 1"/>
-      </material>
-    </visual>
-    <collision>
-      <origin xyz="0 0 0" rpy="0 0 0"/>
-      <geometry>
-        <mesh filename="package://h1_2_inspire_description/meshes/hand_right/right_thumb_2.STL"/>
-      </geometry>
-    </collision>
-  </link>
-  <joint name="right_thumb_2_joint" type="revolute">
+        <mesh filename="package://h1_2_inspire_description/meshes/hand_right/right_thumb_1.STL"/>
+      </geometry>
+      <material name="">
+        <color rgba="1 1 1 1"/>
+      </material>
+    </visual>
+    <collision>
+      <origin xyz="0 0 0" rpy="0 0 0"/>
+      <geometry>
+        <mesh filename="package://h1_2_inspire_description/meshes/hand_right/right_thumb_1.STL"/>
+      </geometry>
+    </collision>
+  </link>
+  <joint name="right_thumb_1_joint" type="revolute">
     <origin xyz="-0.0063016 0.011924 0.003" rpy="1.5708 0 2.7925"/>
-    <parent link="right_thumb_1"/>
-    <child link="right_thumb_2"/>
-    <axis xyz="0 0 1"/>
-    <limit lower="0.035" upper="0.90" effort="1" velocity="100"/>
-  </joint>
-  <link name="right_thumb_3">
+    <parent link="right_thumb_swing"/>
+    <child link="right_thumb_1"/>
+    <axis xyz="0 0 1"/>
+    <limit lower="0" upper="0.92" effort="1" velocity="100"/>
+  </joint>
+  <link name="right_thumb_2">
     <inertial>
       <origin xyz="0.00924505131715823 0.00481918438391222 -0.00753905171750578" rpy="0 0 0"/>
@@ -101,26 +101,26 @@
       <origin xyz="0 0 0" rpy="0 0 0"/>
       <geometry>
-        <mesh filename="package://h1_2_inspire_description/meshes/hand_right/right_thumb_3.STL"/>
-      </geometry>
-      <material name="">
-        <color rgba="1 1 1 1"/>
-      </material>
-    </visual>
-    <collision>
-      <origin xyz="0 0 0" rpy="0 0 0"/>
-      <geometry>
-        <mesh filename="package://h1_2_inspire_description/meshes/hand_right/right_thumb_3.STL"/>
-      </geometry>
-    </collision>
-  </link>
-  <joint name="right_thumb_3_joint" type="revolute">
+        <mesh filename="package://h1_2_inspire_description/meshes/hand_right/right_thumb_2.STL"/>
+      </geometry>
+      <material name="">
+        <color rgba="1 1 1 1"/>
+      </material>
+    </visual>
+    <collision>
+      <origin xyz="0 0 0" rpy="0 0 0"/>
+      <geometry>
+        <mesh filename="package://h1_2_inspire_description/meshes/hand_right/right_thumb_2.STL"/>
+      </geometry>
+    </collision>
+  </link>
+  <joint name="right_thumb_2_joint" type="revolute">
     <origin xyz="0.038292 0.014535 -0.0015" rpy="0 0 0"/>
-    <parent link="right_thumb_2"/>
-    <child link="right_thumb_3"/>
+    <parent link="right_thumb_1"/>
+    <child link="right_thumb_2"/>
     <axis xyz="0 0 1"/>
     <limit lower="0" upper="3.14" effort="1" velocity="100"/>
-    <mimic joint="right_thumb_2_joint" multiplier="0.40" offset="0"/>
-  </joint>
-  <link name="right_thumb_4">
+    <mimic joint="right_thumb_1_joint" multiplier="0.40" offset="0"/>
+  </joint>
+  <link name="right_thumb_3">
     <inertial>
       <origin xyz="0.0136013574986204 0.0105235463357921 -0.00734356571247173" rpy="0 0 0"/>
@@ -132,24 +132,24 @@
       <origin xyz="0 0 0" rpy="0 0 0"/>
       <geometry>
-        <mesh filename="package://h1_2_inspire_description/meshes/hand_right/right_thumb_4.STL"/>
-      </geometry>
-      <material name="">
-        <color rgba="1 1 1 1"/>
-      </material>
-    </visual>
-    <collision>
-      <origin xyz="0 0 0" rpy="0 0 0"/>
-      <geometry>
-        <mesh filename="package://h1_2_inspire_description/meshes/hand_right/right_thumb_4.STL"/>
-      </geometry>
-    </collision>
-  </link>
-  <joint name="right_thumb_4_joint" type="revolute">
+        <mesh filename="package://h1_2_inspire_description/meshes/hand_right/right_thumb_3.STL"/>
+      </geometry>
+      <material name="">
+        <color rgba="1 1 1 1"/>
+      </material>
+    </visual>
+    <collision>
+      <origin xyz="0 0 0" rpy="0 0 0"/>
+      <geometry>
+        <mesh filename="package://h1_2_inspire_description/meshes/hand_right/right_thumb_3.STL"/>
+      </geometry>
+    </collision>
+  </link>
+  <joint name="right_thumb_3_joint" type="revolute">
     <origin xyz="0.018189 0.012576 -0.0002" rpy="0 0 0"/>
-    <parent link="right_thumb_3"/>
-    <child link="right_thumb_4"/>
+    <parent link="right_thumb_2"/>
+    <child link="right_thumb_3"/>
     <axis xyz="0 0 1"/>
     <limit lower="0" upper="3.14" effort="1" velocity="100"/>
-    <mimic joint="right_thumb_2_joint" multiplier="0.60" offset="0"/>
+    <mimic joint="right_thumb_1_joint" multiplier="0.60" offset="0"/>
   </joint>
   <link name="right_index_1">
