Commit message: Mirror the right hand's digits from the left hand
The four fingers matched their mirror to 0.01-1.5 mm but the thumb drifted
from *_thumb_1_joint onward (7.3 -> 18.0 -> 29.0 mm on the link centroids),
because that joint's origin rpy was "1.5708 0 0.037536" on the left and
"1.5708 0 2.7925" on the right -- about 17 degrees off. The two hands came
from separate vendor exports with inconsistent local frame conventions, so
rather than patching one angle, the right hand's digits are now derived from
the left, which is the reference side.

Right digit frames are defined as the exact mirror of the left across the
palm's y=0 plane, frame_right = S * frame_left * S with S = diag(1,-1,1):
  origin xyz  (x,y,z) -> (x,-y,z)
  origin rpy  (r,p,y) -> (-r,p,-y)      [S Rz(y)Ry(p)Rx(r) S = Rz(-y)Ry(p)Rx(-r)]
  axis        (x,y,z) -> (-x,y,-z)      [pseudovector, u -> -S u]
  inertia     ixy, iyz negated          [I' = S I S]
The resulting axes reproduce the values the vendor already had, confirming
the convention. Applied to the 12 digit links and 12 digit joints in both
inspire_hand_right.urdf.xacro and the flat Isaac URDF.

The 12 right digit STL meshes are regenerated as the left meshes with y
negated, swapping v1/v2 per triangle so the winding still matches the
outward normal. Verified: signed volume and normal/winding agreement are
identical to the left (coherence 1.000).

Verification, comparing every mesh vertex in its own palm frame with the
left mirrored in y:
  worst vertex deviation     0.000000 mm  (was up to 28.97 mm on the thumb)
  same joint command on both hands, 6 configurations (open, fully closed,
  thumb-index pinch, 3 random)  0.000000 mm
  thumb tip vs its mirror     0.0000 mm   (was 20.89 mm)
  digit mass, left vs right   0.143381 kg both, difference 0.00e+00

Side effects, both intended consequences of taking the left as reference:
- Right digit masses now come from the left export. The thumb links differ
  most (0.030 -> 0.035, 0.020 -> 0.023, 0.014 -> 0.018 kg); the rest change
  by ~1e-7. Right hand 0.4455 -> 0.4575 kg, robot 61.8499 -> 61.8619 kg.
- Right digits were white (rgba 1 1 1 1) and are now the left's colour. The
  palm was left white by the geometry pass, which looked wrong against its
  own fingers, so its material was aligned too. Cosmetic only.

Out of scope: right_hand_base_link keeps the vendor's own export. Its mesh
is already a good mirror of the left palm (0.05 mm on the centroid), but its
inertial mass is 0.314091 kg against 0.260034 kg on the left, a 54 g gap.
The left export carried a separate flange.STL that the right merges into the
palm, which likely explains it. Not addressed here.

Co-Authored-By: Claude Opus 5 <noreply@anthropic.com>
Claude-Session: https://claude.ai/code/session_01WDAX8VZbrLhjdUkohUZLGo

File: urdf/h1_2_hands_isaac.urdf (robot description, URDF)
Before this commit: robot h1_2_with_inspire_hands, 58 links, 57 joints
Links:
- link right_index_1: mass 0.00719999389753263 -> 0.00719950629120704
- link right_index_2: mass 0.0096859422185797 -> 0.00968687528768598
- link right_little_1: mass 0.00719994987013216 -> 0.00719949424831882
- link right_little_2: mass 0.0075928240732547 -> 0.00759259232694104
- link right_middle_1: mass 0.0071999945469965 -> 0.00719950322487975
- link right_middle_2: mass 0.0104603374244707 -> 0.0104611931926301
- link right_ring_1: mass 0.00719998997814134 -> 0.00719949770218713
- link right_ring_2: mass 0.0096859390369724 -> 0.00968685177133057
- link right_thumb_1: mass 0.030 -> 0.035
- link right_thumb_2: mass 0.020 -> 0.023
- link right_thumb_3: mass 0.014 -> 0.018
Joints:
- joint right_index_1_joint: origin xyz=-0.047006 -0.11125 0.045444 rpy=1.6057 0 -1.5708 -> xyz=-0.048156 -0.11125 0.045404 rpy=-1.6057 0 1.5708
- joint right_index_2_joint: origin xyz=-0.0016312 0.032734 -0.00055 rpy=0 0 0 -> xyz=0.00259487212105013 -0.0326721877470773 -0.000299999999999988 rpy=0 0 0
- joint right_little_1_joint: origin xyz=0.017589 -0.11125 0.042696 rpy=1.4661 0 -1.5708 -> xyz=0.016446 -0.11125 0.042817 rpy=-1.4661 0 1.5708
- joint right_little_2_joint: origin xyz=-0.005182 0.032363 -0.00055 rpy=0 0 1.5708 -> xyz=0.0023072 -0.032694 -0.0003 rpy=0 0 0
- joint right_middle_1_joint: origin xyz=-0.025427 -0.11125 0.046044 rpy=1.5708 0 -1.5708 -> xyz=-0.026577 -0.11125 0.046044 rpy=-1.5708 0 1.5708
- joint right_middle_2_joint: origin xyz=-0.0028436 0.032651 -0.00055 rpy=0 0 0 -> xyz=0.0028436 -0.032651 -0.0003 rpy=0 0 0
- joint right_ring_1_joint: origin xyz=-0.0037966 -0.11125 0.045878 rpy=1.5184 0 -1.5708 -> xyz=-0.004945 -0.11125 0.045939 rpy=-1.5184 0 1.5708
- joint right_ring_2_joint: origin xyz=-0.0031431 0.032624 -0.00055 rpy=0 0 0 -> xyz=0.0031431 -0.032624 -0.0003 rpy=0 0 0
- joint right_thumb_1_joint: origin xyz=-0.0063016 0.011924 0.003 rpy=1.5708 0 2.7925 -> xyz=-0.0096402 0.0097687 0.00125 rpy=-1.5708 0 -0.037536
- joint right_thumb_2_joint: origin xyz=0.038292 0.014535 -0.0015 rpy=0 0 0 -> xyz=-0.0385855343215257 -0.0137354280979689 -0.00085000000007604 rpy=0 0 0
- joint right_thumb_3_joint: origin xyz=0.018189 0.012576 -0.0002 rpy=0 0 0 -> xyz=-0.0204656980659991 -0.00837680232935447 0.000199999999999881 rpy=0 0 0
- joint right_thumb_swing_joint: origin xyz=-0.035227 -0.0908 -0.041956 rpy=0 0 0 -> xyz=-0.035227 -0.0908 -0.040206 rpy=0 0 0

File: urdf/inspire_hand_right.urdf.xacro (robot description, xacro)
@@ -6,5 +6,12 @@
      Mimic joints: right_thumb_2_joint (0.40×), right_thumb_3_joint (0.60×),
        right_index_2_joint (1.05×), right_middle_2_joint (1.05×),
-       right_ring_2_joint (1.05×), right_little_2_joint (1.05×) -->
+       right_ring_2_joint (1.05×), right_little_2_joint (1.05×)
+     The 12 digit links and joints are the EXACT MIRROR of inspire_hand_left
+     across the y=0 plane of the palm: frame_right = S · frame_left · S with
+     S = diag(1,-1,1), so origin xyz (x,y,z) -> (x,-y,z), origin rpy (r,p,y) ->
+     (-r,p,-y), axis (x,y,z) -> (-x,y,-z) and inertia ixy,iyz negated. The
+     meshes in meshes/hand_right/ (except base_link.STL) are the left meshes
+     with y negated. Edit the LEFT hand and re-mirror; do not edit these by
+     hand. right_hand_base_link (the palm) is the vendor's own export. -->
 <robot xmlns:xacro="http://www.ros.org/wiki/xacro">
   <link name="right_hand_base_link">
@@ -21,5 +28,5 @@
       </geometry>
       <material name="">
-        <color rgba="1 1 1 1"/>
+        <color rgba="0.792156862745098 0.819607843137255 0.933333333333333 1"/>
       </material>
     </visual>
@@ -33,8 +40,8 @@
   <link name="right_thumb_swing">
     <inertial>
-      <origin xyz="-0.00178423179132727 0.000649410769092446 0.0048858931043441" rpy="0 0 0"/>
+      <origin xyz="-0.001897403655087 7.12516796909923E-05 0.00313589310434412" rpy="0 0 0"/>
       <mass value="0.00115518743162309"/>
-      <inertia ixx="5.98911473694572E-08" ixy="-8.04324266712912E-09" ixz="-3.29346964287941E-09"
-               iyy="4.07201940087006E-08" iyz="1.1987242259973E-09" izz="6.18161684388651E-08"/>
+      <inertia ixx="6.27834293959477E-08" ixy="-9.38445541803444E-10" ixz="-3.50236810587605E-09"
+               iyy="3.78279141131513E-08" iyz="1.31528360070952E-10" izz="6.1816168438865E-08"/>
     </inertial>
     <visual>
@@ -44,5 +51,5 @@
       </geometry>
       <material name="">
-        <color rgba="1 1 1 1"/>
+        <color rgba="0.792156862745098 0.819607843137255 0.933333333333333 1"/>
       </material>
     </visual>
@@ -55,5 +62,5 @@
   </link>
   <joint name="right_thumb_swing_joint" type="revolute">
-    <origin xyz="-0.035227 -0.0908 -0.041956" rpy="0 0 0"/>
+    <origin xyz="-0.035227 -0.0908 -0.040206" rpy="0 0 0"/>
     <parent link="right_hand_base_link"/>
     <child link="right_thumb_swing"/>
@@ -63,8 +70,8 @@
   <link name="right_thumb_1">
     <inertial>
-      <origin xyz="0.0161097484383394 0.0103028022975375 -0.00905330600289518" rpy="0 0 0"/>
-      <mass value="0.030"/>
-      <inertia ixx="1.05608173707368E-06" ixy="-8.93990422826739E-08" ixz="-4.0717047155279E-10"
-               iyy="1.12055666436187E-06" iyz="-3.12541187909307E-10" izz="1.43604602983943E-06"/>
+      <origin xyz="-0.0163208309809786 -0.00996672794459635 -0.00940273641037634" rpy="0 0 0"/>
+      <mass value="0.035"/>
+      <inertia ixx="1.05252775356938E-06" ixy="-8.8013589531825E-08" ixz="4.12297543062756E-10"
+               iyy="1.12456993863274E-06" iyz="3.58528262599009E-10" izz="1.43633392322177E-06"/>
     </inertial>
     <visual>
@@ -74,5 +81,5 @@
       </geometry>
       <material name="">
-        <color rgba="1 1 1 1"/>
+        <color rgba="0.792156862745098 0.819607843137255 0.933333333333333 1"/>
       </material>
     </visual>
@@ -85,5 +92,5 @@
   </link>
   <joint name="right_thumb_1_joint" type="revolute">
-    <origin xyz="-0.0063016 0.011924 0.003" rpy="1.5708 0 2.7925"/>
+    <origin xyz="-0.0096402 0.0097687 0.00125" rpy="-1.5708 0 -0.037536"/>
     <parent link="right_thumb_swing"/>
     <child link="right_thumb_1"/>
@@ -93,8 +100,8 @@
   <link name="right_thumb_2">
     <inertial>
-      <origin xyz="0.00924505131715823 0.00481918438391222 -0.00753905171750578" rpy="0 0 0"/>
-      <mass value="0.020"/>
-      <inertia ixx="4.84948263631248E-07" ixy="-4.6215685121335E-08" ixz="-5.73077020148322E-11"
-               iyy="3.97628031594582E-07" iyz="-2.99889919786187E-10" izz="4.38765869483229E-07"/>
+      <origin xyz="-0.0100669921030146 -0.0027226860312175 -0.00854141424002414" rpy="0 0 0"/>
+      <mass value="0.023"/>
+      <inertia ixx="4.61650984659959E-07" ixy="-6.02617854200335E-08" ixz="4.49999330286846E-11"
+               iyy="4.2100553287784E-07" iyz="2.1886405983307E-10" izz="4.38695633575155E-07"/>
     </inertial>
     <visual>
@@ -104,5 +111,5 @@
       </geometry>
       <material name="">
-        <color rgba="1 1 1 1"/>
+        <color rgba="0.792156862745098 0.819607843137255 0.933333333333333 1"/>
       </material>
     </visual>
@@ -115,5 +122,5 @@
   </link>
   <joint name="right_thumb_2_joint" type="revolute">
-    <origin xyz="0.038292 0.014535 -0.0015" rpy="0 0 0"/>
+    <origin xyz="-0.0385855343215257 -0.0137354280979689 -0.00085000000007604" rpy="0 0 0"/>
     <parent link="right_thumb_1"/>
     <child link="right_thumb_2"/>
@@ -124,8 +131,8 @@
   <link name="right_thumb_3">
     <inertial>
-      <origin xyz="0.0136013574986204 0.0105235463357921 -0.00734356571247173" rpy="0 0 0"/>
-      <mass value="0.014"/>
-      <inertia ixx="7.90885781861325E-07" ixy="-2.49464441546171E-07" ixz="6.42303183060523E-10"
-               iyy="6.16404813927616E-07" iyz="9.69366750167204E-10" izz="9.25691764995085E-07"/>
+      <origin xyz="-0.0166252667929019 -0.00439732092491903 -0.00874331047569411" rpy="0 0 0"/>
+      <mass value="0.018"/>
+      <inertia ixx="5.85505830748828E-07" ixy="-2.36405978862981E-07" ixz="-9.42185151685949E-10"
+               iyy="8.21798877779441E-07" iyz="-6.15791569450789E-10" izz="9.25701229462772E-07"/>
     </inertial>
     <visual>
@@ -135,5 +142,5 @@
       </geometry>
       <material name="">
-        <color rgba="1 1 1 1"/>
+        <color rgba="0.792156862745098 0.819607843137255 0.933333333333333 1"/>
       </material>
     </visual>
@@ -146,5 +153,5 @@
   </link>
   <joint name="right_thumb_3_joint" type="revolute">
-    <origin xyz="0.018189 0.012576 -0.0002" rpy="0 0 0"/>
+    <origin xyz="-0.0204656980659991 -0.00837680232935447 0.000199999999999881" rpy="0 0 0"/>
     <parent link="right_thumb_2"/>
     <child link="right_thumb_3"/>
@@ -155,8 +162,8 @@
   <link name="right_index_1">
     <inertial>
-      <origin xyz="-0.00183546255523358 0.0123552521861834 -0.00664922294778368" rpy="0 0 0"/>
-      <mass value="0.00719999389753263"/>
-      <inertia ixx="1.28371991025319E-06" ixy="4.21564829206075E-08" ixz="-4.10859703076842E-12"
-               iyy="5.79478432222903E-07" iyz="6.39690407241903E-11" izz="1.32925246769088E-06"/>
+      <origin xyz="0.00219916454162671 -0.0122949545354551 -0.00779931609805271" rpy="0 0 0"/>
+      <mass value="0.00719950629120704"/>
+      <inertia ixx="1.28051762409609E-06" ixy="6.28742259934098E-08" ixz="8.85831478756991E-13"
+               iyy="5.82545787352841E-07" iyz="-8.55749735433038E-11" izz="1.32913319060816E-06"/>
     </inertial>
     <visual>
@@ -166,5 +173,5 @@
       </geometry>
       <material name="">
-        <color rgba="1 1 1 1"/>
+        <color rgba="0.792156862745098 0.819607843137255 0.933333333333333 1"/>
       </material>
     </visual>
@@ -177,5 +184,5 @@
   </link>
   <joint name="right_index_1_joint" type="revolute">
-    <origin xyz="-0.047006 -0.11125 0.045444" rpy="1.6057 0 -1.5708"/>
+    <origin xyz="-0.048156 -0.11125 0.045404" rpy="-1.6057 0 1.5708"/>
     <parent link="right_hand_base_link"/>
     <child link="right_index_1"/>
@@ -185,8 +192,8 @@
   <link name="right_index_2">
     <inertial>
-      <origin xyz="0.000405081354201142 0.0257028143581744 -0.00609275623125877" rpy="0 0 0"/>
-      <mass value="0.0096859422185797"/>
-      <inertia ixx="2.25513837942244E-06" ixy="4.11239564383381E-07" ixz="-3.94499739658712E-10"
-               iyy="3.91290903748666E-07" iyz="2.79706871963247E-09" izz="2.30200483771215E-06"/>
+      <origin xyz="-0.000690175178177488 -0.0256943199737118 -0.0074925254099278" rpy="0 0 0"/>
+      <mass value="0.00968687528768598"/>
+      <inertia ixx="2.26451337650877E-06" ixy="3.90524448356852E-07" ixz="3.56545732231415E-10"
+               iyy="3.82394128669363E-07" iyz="-2.76896757225301E-09" izz="2.302471439937E-06"/>
     </inertial>
     <visual>
@@ -196,5 +203,5 @@
       </geometry>
       <material name="">
-        <color rgba="1 1 1 1"/>
+        <color rgba="0.792156862745098 0.819607843137255 0.933333333333333 1"/>
       </material>
     </visual>
@@ -207,5 +214,5 @@
   </link>
   <joint name="right_index_2_joint" type="revolute">
-    <origin xyz="-0.0016312 0.032734 -0.00055" rpy="0 0 0"/>
+    <origin xyz="0.00259487212105013 -0.0326721877470773 -0.000299999999999988" rpy="0 0 0"/>
     <parent link="right_index_1"/>
     <child link="right_index_2"/>
@@ -216,8 +223,8 @@
   <link name="right_middle_1">
     <inertial>
-      <origin xyz="-0.00229221489529488 0.0122787164691098 -0.00664923691414206" rpy="0 0 0"/>
-      <mass value="0.0071999945469965"/>
-      <inertia ixx="1.27961146095209E-06" ixy="6.81307502326405E-08" ixz="-6.13869092494893E-12"
-               iyy="5.83570383259162E-07" iyz="6.33401074036368E-11" izz="1.32923656099557E-06"/>
+      <origin xyz="0.00229271394242234 -0.0122778605414752 -0.00779931823074317" rpy="0 0 0"/>
+      <mass value="0.00719950322487975"/>
+      <inertia ixx="1.27951858905778E-06" ixy="6.81813021711601E-08" ixz="1.5855112157922E-12"
+               iyy="5.83543537428456E-07" iyz="-8.56179612609339E-11" izz="1.32913234511164E-06"/>
     </inertial>
     <visual>
@@ -227,5 +234,5 @@
       </geometry>
       <material name="">
-        <color rgba="1 1 1 1"/>
+        <color rgba="0.792156862745098 0.819607843137255 0.933333333333333 1"/>
       </material>
     </visual>
@@ -238,5 +245,5 @@
   </link>
   <joint name="right_middle_1_joint" type="revolute">
-    <origin xyz="-0.025427 -0.11125 0.046044" rpy="1.5708 0 -1.5708"/>
+    <origin xyz="-0.026577 -0.11125 0.046044" rpy="-1.5708 0 1.5708"/>
     <parent link="right_hand_base_link"/>
     <child link="right_middle_1"/>
@@ -246,8 +253,8 @@
   <link name="right_middle_2">
     <inertial>
-      <origin xyz="7.55635118059039E-05 0.0274472409648012 -0.00610051224365681" rpy="0 0 0"/>
-      <mass value="0.0104603374244707"/>
-      <inertia ixx="2.75802690508112E-06" ixy="4.66354191476345E-07" ixz="-3.7332807411606E-12"
-               iyy="4.22418749309736E-07" iyz="7.48556574992485E-11" izz="2.8069463787114E-06"/>
+      <origin xyz="-7.51983994427274E-05 -0.027448753770842 -0.00750059894166984" rpy="0 0 0"/>
+      <mass value="0.0104611931926301"/>
+      <inertia ixx="2.75831931773332E-06" ixy="4.66412841401028E-07" ixz="7.3576656177484E-12"
+               iyy="4.22466538741155E-07" iyz="-1.79608426686722E-11" izz="2.80722617348706E-06"/>
     </inertial>
     <visual>
@@ -257,5 +264,5 @@
       </geometry>
       <material name="">
-        <color rgba="1 1 1 1"/>
+        <color rgba="0.792156862745098 0.819607843137255 0.933333333333333 1"/>
       </material>
     </visual>
@@ -268,5 +275,5 @@
   </link>
   <joint name="right_middle_2_joint" type="revolute">
-    <origin xyz="-0.0028436 0.032651 -0.00055" rpy="0 0 0"/>
+    <origin xyz="0.0028436 -0.032651 -0.0003" rpy="0 0 0"/>
     <parent link="right_middle_1"/>
     <child link="right_middle_2"/>
@@ -277,8 +284,8 @@
   <link name="right_ring_1">
     <inertial>
-      <origin xyz="-0.00240481178777663 0.0122571709475593 -0.00664923625225445" rpy="0 0 0"/>
-      <mass value="0.00719998997814134"/>
-      <inertia ixx="1.27830103769765E-06" ixy="7.45073064952644E-08" ixz="-6.73880804378546E-12"
-               iyy="5.84879553082369E-07" iyz="6.33505850524704E-11" izz="1.32923557625194E-06"/>
+      <origin xyz="0.00240530428455067 -0.0122563079467745 -0.00779931923444504" rpy="0 0 0"/>
+      <mass value="0.00719949770218713"/>
+      <inertia ixx="1.27820682409824E-06" ixy="7.45572429780095E-08" ixz="2.25718181777012E-12"
+               iyy="5.84853511073516E-07" iyz="-8.5622233041164E-11" izz="1.32913088941838E-06"/>
     </inertial>
     <visual>
@@ -288,5 +295,5 @@
       </geometry>
       <material name="">
-        <color rgba="1 1 1 1"/>
+        <color rgba="0.792156862745098 0.819607843137255 0.933333333333333 1"/>
       </material>
     </visual>
@@ -299,5 +306,5 @@
   </link>
   <joint name="right_ring_1_joint" type="revolute">
-    <origin xyz="-0.0037966 -0.11125 0.045878" rpy="1.5184 0 -1.5708"/>
+    <origin xyz="-0.004945 -0.11125 0.045939" rpy="-1.5184 0 1.5708"/>
     <parent link="right_hand_base_link"/>
     <child link="right_ring_1"/>
@@ -307,8 +314,8 @@
   <link name="right_ring_2">
     <inertial>
-      <origin xyz="0.000666830906754845 0.0256973412492289 -0.0060927714564012" rpy="0 0 0"/>
-      <mass value="0.0096859390369724"/>
-      <inertia ixx="2.26332196405867E-06" ixy="3.92172318180451E-07" ixz="-3.6571544042072E-10"
-               iyy="3.83108005467821E-07" iyz="2.80158649618188E-09" izz="2.30200501593561E-06"/>
+      <origin xyz="-0.000667145407605998 -0.0256949163202511 -0.00749252997688842" rpy="0 0 0"/>
+      <mass value="0.00968685177133057"/>
+      <inertia ixx="2.26381138740299E-06" ixy="3.92210300202205E-07" ixz="3.58404653503586E-10"
+               iyy="3.83095000534084E-07" iyz="-2.77027363965472E-09" izz="2.30247104599333E-06"/>
     </inertial>
     <visual>
@@ -318,5 +325,5 @@
       </geometry>
       <material name="">
-        <color rgba="1 1 1 1"/>
+        <color rgba="0.792156862745098 0.819607843137255 0.933333333333333 1"/>
       </material>
     </visual>
@@ -329,5 +336,5 @@
   </link>
   <joint name="right_ring_2_joint" type="revolute">
-    <origin xyz="-0.0031431 0.032624 -0.00055" rpy="0 0 0"/>
+    <origin xyz="0.0031431 -0.032624 -0.0003" rpy="0 0 0"/>
     <parent link="right_ring_1"/>
     <child link="right_ring_2"/>
@@ -338,8 +345,8 @@
   <link name="right_little_1">
     <inertial>
-      <origin xyz="-0.00316844591541322 0.0120823779446085 -0.00664923024026526" rpy="0 0 0"/>
-      <mass value="0.00719994987013216"/>
-      <inertia ixx="1.26624415714453E-06" ixy="1.17303714016617E-07" ixz="-1.15327375315847E-11"
-               iyy="5.96925804604496E-07" iyz="6.36110319317551E-11" izz="1.32922857962207E-06"/>
+      <origin xyz="0.0020908902145567 -0.0123138388094518 -0.00779930416612102" rpy="0 0 0"/>
+      <mass value="0.00719949424831882"/>
+      <inertia ixx="1.28158473132988E-06" ixy="5.67213995105241E-08" ixz="3.81932384005559E-13"
+               iyy="5.81492545898195E-07" iyz="-8.62730752553906E-11" izz="1.32914698853052E-06"/>
     </inertial>
     <visual>
@@ -349,5 +356,5 @@
       </geometry>
       <material name="">
-        <color rgba="1 1 1 1"/>
+        <color rgba="0.792156862745098 0.819607843137255 0.933333333333333 1"/>
       </material>
     </visual>
@@ -360,5 +367,5 @@
   </link>
   <joint name="right_little_1_joint" type="revolute">
-    <origin xyz="0.017589 -0.11125 0.042696" rpy="1.4661 0 -1.5708"/>
+    <origin xyz="0.016446 -0.11125 0.042817" rpy="-1.4661 0 1.5708"/>
     <parent link="right_hand_base_link"/>
     <child link="right_little_1"/>
@@ -368,8 +375,8 @@
   <link name="right_little_2">
     <inertial>
-      <origin xyz="0.0204417303421136 -0.00469494170410353 -0.00609999668427265" rpy="0 0 0"/>
-      <mass value="0.0075928240732547"/>
-      <inertia ixx="2.31546812157118E-07" ixy="-7.27021381773956E-08" ixz="2.36649664862442E-11"
-               iyy="1.27663957628266E-06" iyz="-7.58283070676227E-12" izz="1.23909562166535E-06"/>
+      <origin xyz="-0.0017604035921492 -0.0209002097557272 -0.00750031127302827" rpy="0 0 0"/>
+      <mass value="0.00759259232694104"/>
+      <inertia ixx="1.2354235368985E-06" ixy="2.15945048600066E-07" ixz="3.12205526892557E-12"
+               iyy="2.72718801980276E-07" iyz="-1.27574096139233E-11" izz="1.23906813966421E-06"/>
     </inertial>
     <visual>
@@ -379,5 +386,5 @@
       </geometry>
       <material name="">
-        <color rgba="1 1 1 1"/>
+        <color rgba="0.792156862745098 0.819607843137255 0.933333333333333 1"/>
       </material>
     </visual>
@@ -390,5 +397,5 @@
   </link>
   <joint name="right_little_2_joint" type="revolute">
-    <origin xyz="-0.005182 0.032363 -0.00055" rpy="0 0 1.5708"/>
+    <origin xyz="0.0023072 -0.032694 -0.0003" rpy="0 0 0"/>
     <parent link="right_little_1"/>
     <child link="right_little_2"/>
