Commit message: Include the wrist flange in both palm inertials
Both hands now declare the same palm inertial, 0.314091 kg, which accounts
for the wrist flange that the real RH56DFTP carries. The flange stays out of
the visual and collision model.

The left palm declared 0.260034 kg and the right 0.314091 kg, a 54.06 g gap.
The left export shipped a separate flange.STL (removed in 0bc5cfd as an
unused mesh) that the right appears to fold into the palm, which accounts for
the difference, so 0.314091 kg is the with-flange figure and is now used on
both sides.

The right palm's inertial could not be used as the source. Its declared centre
of mass sits 162.5 mm away from the centroid of its own mesh, i.e. in a
different frame altogether, while the left palm's matches its mesh centroid to
0.0 mm. So the values are built from the left palm and mirrored to the right,
which also repairs that pre-existing defect.

Where the flange seats on the palm is not recoverable from the vendor files:
flange.STL is a bare 75 mm disc in its own frame, in millimetres, and it is
wider than the palm's 50 mm wrist stem, so it cannot be located by fitting.
A guessed lever arm would not be harmless -- at a plausible ~6 cm the Steiner
term m*d^2 is 2.1e-4 kg m^2, about the size of the palm's entire tensor. The
54 g is therefore spread like the rest of the palm instead: centre of mass
unchanged, tensor scaled by 0.314091/0.260034 = 1.207882. This is stated in
both hand headers and in the README.

Verification:
  palm inertial, left vs right   exact mirror: com, mass and tensor
  hand mass, left vs right       0.457472 kg both
  robot total                    61.8619 -> 61.9159 kg
  palm + digits vs the mirror    0.000000 mm
  inertia tensors                51 bodies, all positive definite and
                                 satisfying the triangle inequality
  XML 7/7, xacro 3/3, check_urdf 4/4, loads in Pinocchio

Co-Authored-By: Claude Opus 5 <noreply@anthropic.com>
Claude-Session: https://claude.ai/code/session_01WDAX8VZbrLhjdUkohUZLGo

File: urdf/h1_2_hands_isaac.urdf (robot description, URDF)
Before this commit: robot h1_2_with_inspire_hands, 58 links, 57 joints
Links:
- link left_hand_base_link: mass 0.260034351027079 -> 0.314090908651444

File: urdf/inspire_hand_left.urdf.xacro (robot description, xacro)
@@ -6,12 +6,20 @@
      Mimic joints: left_thumb_2_joint (0.40×), left_thumb_3_joint (0.60×),
        left_index_2_joint (1.05×), left_middle_2_joint (1.05×),
-       left_ring_2_joint (1.05×), left_little_2_joint (1.05×) -->
+       left_ring_2_joint (1.05×), left_little_2_joint (1.05×)
+     The palm's inertial includes the wrist flange (the part shipped as the
+     old meshes/hand_left/flange.STL): 0.260034 kg of palm + 0.054057 kg of
+     flange = 0.314091 kg. The flange is NOT in the visual or collision model.
+     Its exact seat on the palm is unknown: its mesh is a bare 75 mm disc in
+     its own frame, wider than the palm's wrist stem, so rather than invent a
+     lever arm, the 54 g is spread like the rest of the palm: the centre of
+     mass is unchanged and the tensor is scaled by 0.314091/0.260034 = 1.207882.
+     Both palms carry the same values, mirrored. -->
 <robot xmlns:xacro="http://www.ros.org/wiki/xacro">
   <link name="left_hand_base_link">
     <inertial>
       <origin xyz="-0.00826856171690858 0.115495645683634 -0.0283405186091888" rpy="0 0 0"/>
-      <mass value="0.260034351027079"/>
-      <inertia ixx="0.000223659755568991" ixy="1.13436481431654E-06" ixz="5.34309330483412E-07"
-               iyy="0.000266799681382808" iyz="-1.40944118439409E-05" izz="0.00013285776917007"/>
+      <mass value="0.314090908651444"/>
+      <inertia ixx="0.000270154676018588" ixy="1.37017926233064E-06" ixz="6.45382821345028E-07"
+               iyy="0.0003222626319271" iyz="-1.70243916062846E-05" izz="0.000160476557328711"/>
     </inertial>
     <visual>

File: urdf/inspire_hand_right.urdf.xacro (robot description, xacro)
@@ -13,12 +13,20 @@
      meshes in meshes/hand_right/ (except base_link.STL) are the left meshes
      with y negated. Edit the LEFT hand and re-mirror; do not edit these by
-     hand. right_hand_base_link (the palm) is the vendor's own export. -->
+     hand. right_hand_base_link (the palm) is the vendor's own export.
+     The palm's inertial includes the wrist flange (the part shipped as the
+     old meshes/hand_left/flange.STL): 0.260034 kg of palm + 0.054057 kg of
+     flange = 0.314091 kg. The flange is NOT in the visual or collision model.
+     Its exact seat on the palm is unknown: its mesh is a bare 75 mm disc in
+     its own frame, wider than the palm's wrist stem, so rather than invent a
+     lever arm, the 54 g is spread like the rest of the palm: the centre of
+     mass is unchanged and the tensor is scaled by 0.314091/0.260034 = 1.207882.
+     Both palms carry the same values, mirrored. -->
 <robot xmlns:xacro="http://www.ros.org/wiki/xacro">
   <link name="right_hand_base_link">
     <inertial>
-      <origin xyz="-0.00827757758571113 -0.0384721010257447 0.114789391580906" rpy="0 0 0"/>
+      <origin xyz="-0.00826856171690858 -0.115495645683634 -0.0283405186091888" rpy="0 0 0"/>
       <mass value="0.314090908651444"/>
-      <inertia ixx="0.000240584294377349" ixy="5.34716372850393E-07" ixz="1.12900344118066E-06"
-               iyy="0.000155854672232219" iyz="-1.41174523865224E-05" izz="0.000284423438512345"/>
+      <inertia ixx="0.000270154676018588" ixy="-1.37017926233064E-06" ixz="6.45382821345028E-07"
+               iyy="0.0003222626319271" iyz="1.70243916062846E-05" izz="0.000160476557328711"/>
     </inertial>
     <visual>

Commit message: Set hand mass from a scale reading: 0.840 kg per hand
The hand weighed 0.840 kg on a scale, wrist flange included, against 0.457472
kg in the model. The gap is an export artefact, not a modelling choice: the
CAD was never given real materials. Implied densities per link come out as

  palm, *_thumb_swing, all eight finger phalanges   ~1000 kg/m3
  *_thumb_1, *_thumb_2                              5370, 5660 kg/m3
  *_thumb_3                                         1976 kg/m3

so every link except the three hand-edited thumb ones sits at SolidWorks'
default 1000 kg/m3, and the exported 457 g was never a measurement.

The missing 382.528 g goes entirely to the palm, which now carries
0.840 - 0.143381 = 0.696619 kg. The digits are left alone. Reasons:
- The palm holds the six actuators, gearboxes, controller and wiring, which
  is exactly the content a materials-free export leaves out.
- It puts the palm at 2682 kg/m3, an aluminium housing packed with motors.
- Scaling the whole hand by 1.8362 instead would drive *_thumb_1 and
  *_thumb_2 to 9900 and 10400 kg/m3, denser than steel and near lead. Not
  physical.
- Inflating the phalanges by 84% would distort fingertip inertia, which is
  what contact and teleoperation actually depend on.

Centre of mass unchanged, tensor scaled by 0.696619/0.314091 = 2.217891,
preserving the vendor's mass distribution. That distribution is 0.52-0.75x a
homogeneous solid of the same mass, i.e. concentrated toward the centre,
which is what motors and gearboxes in the middle of a palm should look like,
so scaling it is the right way to add more of the same.

Verification:
  hand mass, each side          0.840000000 kg exactly
  robot total                   68.664000 kg = 66.9840 + 2 x 0.840
  inertia tensors               51 bodies, all positive definite and
                                satisfying the triangle inequality
  palm realizability            I_max 7.187e-04 <= m*R^2 5.308e-03, 13.5% of
                                the bound, R measured from the com to the
                                farthest mesh vertex
  left vs right                 exact mirror in com, mass and tensor on all
                                13 links per hand
  geometry                      untouched, asymmetry still 0.000000 mm
  XML 7/7, xacro 3/3, check_urdf 4/4

README and both hand headers updated, including the Pinocchio fixed-base
figure, which is now 62.6810 kg.

Co-Authored-By: Claude Opus 5 <noreply@anthropic.com>
Claude-Session: https://claude.ai/code/session_01WDAX8VZbrLhjdUkohUZLGo

File: urdf/h1_2_hands_isaac.urdf (robot description, URDF)
Before this commit: robot h1_2_with_inspire_hands, 58 links, 57 joints
Links:
- link left_hand_base_link: mass 0.314090908651444 -> 0.696619298523196
- link right_hand_base_link: mass 0.314090908651444 -> 0.696619298523196

File: urdf/inspire_hand_left.urdf.xacro (robot description, xacro)
@@ -7,19 +7,20 @@
        left_index_2_joint (1.05×), left_middle_2_joint (1.05×),
        left_ring_2_joint (1.05×), left_little_2_joint (1.05×)
-     The palm's inertial includes the wrist flange (the part shipped as the
-     old meshes/hand_left/flange.STL): 0.260034 kg of palm + 0.054057 kg of
-     flange = 0.314091 kg. The flange is NOT in the visual or collision model.
-     Its exact seat on the palm is unknown: its mesh is a bare 75 mm disc in
-     its own frame, wider than the palm's wrist stem, so rather than invent a
-     lever arm, the 54 g is spread like the rest of the palm: the centre of
-     mass is unchanged and the tensor is scaled by 0.314091/0.260034 = 1.207882.
-     Both palms carry the same values, mirrored. -->
+     Palm mass is set from a scale reading of the real hand: 0.840 kg for the
+     whole hand, wrist flange included. The 12 digits keep their exported
+     0.143381 kg, so the palm carries 0.840 - 0.143381 = 0.696619 kg. The
+     deficit went to the palm because that is where the six actuators, the
+     gearboxes, the controller and the wiring sit, and because the CAD export
+     left almost every link at SolidWorks' default 1000 kg/m3. The flange is
+     NOT in the visual or collision model. The centre of mass is unchanged and
+     the tensor is scaled by 0.696619/0.314091 = 2.217891, which keeps the
+     vendor's mass distribution. Both palms carry the same values, mirrored. -->
 <robot xmlns:xacro="http://www.ros.org/wiki/xacro">
   <link name="left_hand_base_link">
     <inertial>
       <origin xyz="-0.00826856171690858 0.115495645683634 -0.0283405186091888" rpy="0 0 0"/>
-      <mass value="0.314090908651444"/>
-      <inertia ixx="0.000270154676018588" ixy="1.37017926233064E-06" ixz="6.45382821345028E-07"
-               iyy="0.0003222626319271" iyz="-1.70243916062846E-05" izz="0.000160476557328711"/>
+      <mass value="0.696619298523196"/>
+      <inertia ixx="0.000599173537715081" ixy="3.03890781389993E-06" ixz="1.43138854357359E-06"
+               iyy="0.000714743287404168" iyz="-3.77582394519895E-05" izz="0.000355919460629158"/>
     </inertial>
     <visual>

File: urdf/inspire_hand_right.urdf.xacro (robot description, xacro)
@@ -14,19 +14,20 @@
      with y negated. Edit the LEFT hand and re-mirror; do not edit these by
      hand. right_hand_base_link (the palm) is the vendor's own export.
-     The palm's inertial includes the wrist flange (the part shipped as the
-     old meshes/hand_left/flange.STL): 0.260034 kg of palm + 0.054057 kg of
-     flange = 0.314091 kg. The flange is NOT in the visual or collision model.
-     Its exact seat on the palm is unknown: its mesh is a bare 75 mm disc in
-     its own frame, wider than the palm's wrist stem, so rather than invent a
-     lever arm, the 54 g is spread like the rest of the palm: the centre of
-     mass is unchanged and the tensor is scaled by 0.314091/0.260034 = 1.207882.
-     Both palms carry the same values, mirrored. -->
+     Palm mass is set from a scale reading of the real hand: 0.840 kg for the
+     whole hand, wrist flange included. The 12 digits keep their exported
+     0.143381 kg, so the palm carries 0.840 - 0.143381 = 0.696619 kg. The
+     deficit went to the palm because that is where the six actuators, the
+     gearboxes, the controller and the wiring sit, and because the CAD export
+     left almost every link at SolidWorks' default 1000 kg/m3. The flange is
+     NOT in the visual or collision model. The centre of mass is unchanged and
+     the tensor is scaled by 0.696619/0.314091 = 2.217891, which keeps the
+     vendor's mass distribution. Both palms carry the same values, mirrored. -->
 <robot xmlns:xacro="http://www.ros.org/wiki/xacro">
   <link name="right_hand_base_link">
     <inertial>
       <origin xyz="-0.00826856171690858 -0.115495645683634 -0.0283405186091888" rpy="0 0 0"/>
-      <mass value="0.314090908651444"/>
-      <inertia ixx="0.000270154676018588" ixy="-1.37017926233064E-06" ixz="6.45382821345028E-07"
-               iyy="0.0003222626319271" iyz="1.70243916062846E-05" izz="0.000160476557328711"/>
+      <mass value="0.696619298523196"/>
+      <inertia ixx="0.000599173537715081" ixy="-3.03890781389993E-06" ixz="1.43138854357359E-06"
+               iyy="0.000714743287404168" iyz="3.77582394519895E-05" izz="0.000355919460629158"/>
     </inertial>
     <visual>
